File: main_board4.kicad_pcb (KiCad board)
At the start: 2 copper layers, 320 x 140 mm, 84 parts

Commit message: working on pcb layout
Parts:
- added D1: DIODE, Diode_SMD:D_MiniMELF, F.Cu at (448.0, 141.6)
- added D10: DIODE, Diode_SMD:D_MiniMELF, F.Cu at (448.0, 148.4)
- added D11: DIODE, Diode_SMD:D_MiniMELF, F.Cu at (561.6, 69.2)
- added D12: DIODE, Diode_SMD:D_MiniMELF, F.Cu at (458.7, 141.6)
- added D13: DIODE, Diode_SMD:D_MiniMELF, F.Cu at (453.4, 146.1)
- added D14: DIODE, Diode_SMD:D_MiniMELF, F.Cu at (490.8, 140.9)
- added D15: DIODE, Diode_SMD:D_MiniMELF, F.Cu at (458.7, 143.9)
- added D16: DIODE, Diode_SMD:D_MiniMELF, F.Cu at (448.0, 143.9)
- added D17: DIODE, Diode_SMD:D_MiniMELF, F.Cu at (512.2, 147.6)
- added D18: DIODE, Diode_SMD:D_MiniMELF, F.Cu at (517.6, 143.1)
- added D19: DIODE, Diode_SMD:D_MiniMELF, F.Cu at (453.4, 148.4)
- added D2: DIODE, Diode_SMD:D_MiniMELF, F.Cu at (442.7, 143.9)
- added D20: DIODE, Diode_SMD:D_MiniMELF, F.Cu at (517.6, 147.6)
- added D21: DIODE, Diode_SMD:D_MiniMELF, F.Cu at (522.9, 147.6)
- added D22: DIODE, Diode_SMD:D_MiniMELF, F.Cu at (474.8, 146.1)
- added D23: DIODE, Diode_SMD:D_MiniMELF, F.Cu at (567.0, 69.2)
- added D24: DIODE, Diode_SMD:D_MiniMELF, F.Cu at (464.1, 146.1)
- added D25: DIODE, Diode_SMD:D_MiniMELF, F.Cu at (458.7, 148.4)
- added D26: DIODE, Diode_SMD:D_MiniMELF, F.Cu at (464.1, 143.9)
- added D27: DIODE, Diode_SMD:D_MiniMELF, F.Cu at (469.4, 143.1)
- added D28: DIODE, Diode_SMD:D_MiniMELF, F.Cu at (458.7, 146.1)
- added D29: DIODE, Diode_SMD:D_MiniMELF, F.Cu at (464.1, 148.4)
- added D3: DIODE, Diode_SMD:D_MiniMELF, F.Cu at (485.4, 140.9)
- added D30: DIODE, Diode_SMD:D_MiniMELF, F.Cu at (474.8, 141.6)
- added D31: DIODE, Diode_SMD:D_MiniMELF, F.Cu at (469.4, 147.6)
- added D32: DIODE, Diode_SMD:D_MiniMELF, F.Cu at (480.1, 143.1)
- added D33: DIODE, Diode_SMD:D_MiniMELF, F.Cu at (464.1, 141.6)
- added D34: DIODE, Diode_SMD:D_MiniMELF, F.Cu at (469.4, 145.4)
- added D35: DIODE, Diode_SMD:D_MiniMELF, F.Cu at (480.1, 145.4)
- added D36: DIODE, Diode_SMD:D_MiniMELF, F.Cu at (485.5, 143.1)
- added D37: DIODE, Diode_SMD:D_MiniMELF, F.Cu at (485.5, 145.4)
- added D38: DIODE, Diode_SMD:D_MiniMELF, F.Cu at (480.1, 147.6)
- added D39: DIODE, Diode_SMD:D_MiniMELF, F.Cu at (485.5, 147.6)
- added D4: DIODE, Diode_SMD:D_MiniMELF, F.Cu at (442.7, 141.6)
- added D40: DIODE, Diode_SMD:D_MiniMELF, F.Cu at (474.8, 148.4)
- added D41: DIODE, Diode_SMD:D_MiniMELF, F.Cu at (496.1, 140.9)
- added D42: DIODE, Diode_SMD:D_MiniMELF, F.Cu at (490.8, 143.1)
- added D43: DIODE, Diode_SMD:D_MiniMELF, F.Cu at (490.8, 145.4)
- added D44: DIODE, Diode_SMD:D_MiniMELF, F.Cu at (572.3, 69.2)
- added D45: DIODE, Diode_SMD:D_MiniMELF, F.Cu at (474.8, 143.9)
- added D46: DIODE, Diode_SMD:D_MiniMELF, F.Cu at (453.4, 143.9)
- added D47: DIODE, Diode_SMD:D_MiniMELF, F.Cu at (496.2, 145.4)
- added D48: DIODE, Diode_SMD:D_MiniMELF, F.Cu at (501.5, 140.9)
- added D49: DIODE, Diode_SMD:D_MiniMELF, F.Cu at (506.9, 140.9)
- added D5: DIODE, Diode_SMD:D_MiniMELF, F.Cu at (442.7, 146.1)
- added D50: DIODE, Diode_SMD:D_MiniMELF, F.Cu at (512.2, 140.9)
- added D51: DIODE, Diode_SMD:D_MiniMELF, F.Cu at (517.6, 140.9)
- added D52: DIODE, Diode_SMD:D_MiniMELF, F.Cu at (522.9, 140.9)
- added D53: DIODE, Diode_SMD:D_MiniMELF, F.Cu at (528.3, 140.9)
- added D54: DIODE, Diode_SMD:D_MiniMELF, F.Cu at (501.5, 143.1)
- added D55: DIODE, Diode_SMD:D_MiniMELF, F.Cu at (506.9, 143.1)
- added D56: DIODE, Diode_SMD:D_MiniMELF, F.Cu at (512.2, 143.1)
- added D57: DIODE, Diode_SMD:D_MiniMELF, F.Cu at (496.2, 143.1)
- added D58: DIODE, Diode_SMD:D_MiniMELF, F.Cu at (490.8, 147.6)
- added D59: DIODE, Diode_SMD:D_MiniMELF, F.Cu at (522.9, 143.1)
- added D6: DIODE, Diode_SMD:D_MiniMELF, F.Cu at (453.4, 141.6)
- added D60: DIODE, Diode_SMD:D_MiniMELF, F.Cu at (528.3, 143.1)
- added D61: DIODE, Diode_SMD:D_MiniMELF, F.Cu at (501.5, 145.4)
- added D62: DIODE, Diode_SMD:D_MiniMELF, F.Cu at (506.9, 145.4)
- added D63: DIODE, Diode_SMD:D_MiniMELF, F.Cu at (512.2, 145.4)
- added D64: DIODE, Diode_SMD:D_MiniMELF, F.Cu at (517.6, 145.4)
- added D65: DIODE, Diode_SMD:D_MiniMELF, F.Cu at (522.9, 145.4)
- added D66: DIODE, Diode_SMD:D_MiniMELF, F.Cu at (528.3, 145.4)
- added D67: DIODE, Diode_SMD:D_MiniMELF, F.Cu at (496.2, 147.6)
- added D68: DIODE, Diode_SMD:D_MiniMELF, F.Cu at (501.5, 147.6)
- added D69: DIODE, Diode_SMD:D_MiniMELF, F.Cu at (582.1, 93.6)
- added D7: DIODE, Diode_SMD:D_MiniMELF, F.Cu at (448.0, 146.1)
- added D70: DIODE, Diode_SMD:D_MiniMELF, F.Cu at (583.0, 69.2)
- added D71: DIODE, Diode_SMD:D_MiniMELF, F.Cu at (588.4, 69.2)
- added D72: DIODE, Diode_SMD:D_MiniMELF, F.Cu at (612.8, 53.4)
- added D73: DIODE, Diode_SMD:D_MiniMELF, F.Cu at (612.8, 55.6)
- added D74: DIODE, Diode_SMD:D_MiniMELF, F.Cu at (612.8, 57.9)
- added D75: DIODE, Diode_SMD:D_MiniMELF, F.Cu at (612.8, 60.1)
- added D76: DIODE, Diode_SMD:D_MiniMELF, F.Cu at (576.7, 91.3)
- added D77: DIODE, Diode_SMD:D_MiniMELF, F.Cu at (506.9, 147.6)
- added D78: DIODE, Diode_SMD:D_MiniMELF, F.Cu at (576.7, 93.6)
- added D79: DIODE, Diode_SMD:D_MiniMELF, F.Cu at (576.7, 95.8)
- added D8: DIODE, Diode_SMD:D_MiniMELF, F.Cu at (442.7, 148.4)
- added D80: DIODE, Diode_SMD:D_MiniMELF, F.Cu at (551.9, 129.2)
- added D81: DIODE, Diode_SMD:D_MiniMELF, F.Cu at (577.7, 69.2)
- added D82: DIODE, Diode_SMD:D_MiniMELF, F.Cu at (576.7, 98.1)
- added D83: DIODE, Diode_SMD:D_MiniMELF, F.Cu at (587.4, 91.3)
- added D84: DIODE, Diode_SMD:D_MiniMELF, F.Cu at (582.1, 91.3)
- added D9: DIODE, Diode_SMD:D_MiniMELF, F.Cu at (612.8, 51.1)
- added MCU1: Teensy2.0++, sw_fprint_wLed:Teensy2.0++_footprint_assigned, F.Cu at (198.1, 15.3)
- added P_jump_trans1: CONN_01X01, Connector_PinHeader_2.54mm:PinHeader_1x01_P2.54mm_Vertical, F.Cu at (581.2, 96.5)
- added P_jump_trans2: CONN_01X01, Connector_PinHeader_2.54mm:PinHeader_1x01_P2.54mm_Vertical, F.Cu at (575.9, 101.0)
- added P_jump_trans3: CONN_01X01, Connector_PinHeader_2.54mm:PinHeader_1x01_P2.54mm_Vertical, F.Cu at (611.9, 63.1)
- added R1: R, Resistor_SMD:R_0805_2012Metric, F.Cu at (532.7, 144.6)
- added R10: R, Resistor_SMD:R_0805_2012Metric, F.Cu at (530.7, 148.5)
- added R11: R, Resistor_SMD:R_0805_2012Metric, F.Cu at (615.4, 62.2)
- added R12: R, Resistor_SMD:R_0805_2012Metric, F.Cu at (581.1, 99.3)
- added R13: R, Resistor_SMD:R_0805_2012Metric, F.Cu at (591.8, 91.2)
- added R14: R, Resistor_SMD:R_0805_2012Metric, F.Cu at (579.4, 101.3)
- added R15: R, Resistor_SMD:R_0805_2012Metric, F.Cu at (584.7, 97.6)
- added R16: R, Resistor_SMD:R_0805_2012Metric, F.Cu at (534.1, 148.5)
- added R17: R, Resistor_SMD:R_0805_2012Metric, F.Cu at (579.4, 103.2)
- added R18: R, Resistor_SMD:R_0805_2012Metric, F.Cu at (536.1, 146.6)
- added R19: R, Resistor_SMD:R_0805_2012Metric, F.Cu at (550.9, 131.3)
- added R2: R, Resistor_SMD:R_0805_2012Metric, F.Cu at (536.1, 140.7)
- added R20: R, Resistor_SMD:R_0805_2012Metric, F.Cu at (591.6, 97.3)
- added R21: R, Resistor_SMD:R_0805_2012Metric, F.Cu at (546.3, 142.7)
- added R22: R, Resistor_SMD:R_0805_2012Metric, F.Cu at (550.9, 133.3)
- added R23: R, Resistor_SMD:R_0805_2012Metric, F.Cu at (575.7, 105.8)
- added R24: R, Resistor_SMD:R_0805_2012Metric, F.Cu at (586.4, 93.4)
- added R25: R, Resistor_SMD:R_0805_2012Metric, F.Cu at (556.3, 129.1)
- added R26: R, Resistor_SMD:R_0805_2012Metric, F.Cu at (589.8, 93.4)
- added R27: R, Resistor_SMD:R_0805_2012Metric, F.Cu at (579.1, 105.2)
- added R28: R, Resistor_SMD:R_0805_2012Metric, F.Cu at (575.7, 107.7)
- added R29: R, Resistor_SMD:R_0805_2012Metric, F.Cu at (539.5, 144.6)
- added R3: R, Resistor_SMD:R_0805_2012Metric, F.Cu at (611.8, 65.9)
- added R30: R, Resistor_SMD:R_0805_2012Metric, F.Cu at (584.5, 99.6)
- added R31: R, Resistor_SMD:R_0805_2012Metric, F.Cu at (588.1, 95.4)
- added R32: R, Resistor_SMD:R_0805_2012Metric, F.Cu at (542.9, 140.7)
- added R33: R, Resistor_SMD:R_0805_2012Metric, F.Cu at (539.5, 142.7)
- added R34: R, Resistor_SMD:R_0805_2012Metric, F.Cu at (557.7, 133.0)
- added R35: R, Resistor_SMD:R_0805_2012Metric, F.Cu at (594.8, 88.0)
- added R36: R, Resistor_SMD:R_0805_2012Metric, F.Cu at (598.2, 88.0)
- added R37: R, Resistor_SMD:R_0805_2012Metric, F.Cu at (550.9, 135.2)
- added R38: R, Resistor_SMD:R_0805_2012Metric, F.Cu at (554.3, 131.3)
- added R39: R, Resistor_SMD:R_0805_2012Metric, F.Cu at (546.3, 140.7)
- added R4: R, Resistor_SMD:R_0805_2012Metric, F.Cu at (575.7, 103.8)
- added R40: R, Resistor_SMD:R_0805_2012Metric, F.Cu at (542.9, 142.7)
- added R41: R, Resistor_SMD:R_0805_2012Metric, F.Cu at (542.9, 144.6)
- added R42: R, Resistor_SMD:R_0805_2012Metric, F.Cu at (591.6, 95.4)
- added R43: R, Resistor_SMD:R_0805_2012Metric, F.Cu at (536.1, 144.6)
- added R44: R, Resistor_SMD:R_0805_2012Metric, F.Cu at (527.3, 149.4)
- added R45: R, Resistor_SMD:R_0805_2012Metric, F.Cu at (532.7, 142.7)
- added R46: R, Resistor_SMD:R_0805_2012Metric, F.Cu at (584.7, 95.7)
- added R47: R, Resistor_SMD:R_0805_2012Metric, F.Cu at (582.8, 101.5)
- added R48: R, Resistor_SMD:R_0805_2012Metric, F.Cu at (582.8, 103.5)
- added R49: R, Resistor_SMD:R_0805_2012Metric, F.Cu at (539.5, 146.6)
- added R5: R, Resistor_SMD:R_0805_2012Metric, F.Cu at (615.2, 65.9)
- added R50: R, Resistor_SMD:R_0805_2012Metric, F.Cu at (579.1, 107.1)
- added R51: R, Resistor_SMD:R_0805_2012Metric, F.Cu at (575.7, 109.7)
- added R52: R, Resistor_SMD:R_0805_2012Metric, F.Cu at (575.7, 111.6)
- added R53: R, Resistor_SMD:R_0805_2012Metric, F.Cu at (593.3, 93.1)
- added R54: R, Resistor_SMD:R_0805_2012Metric, F.Cu at (537.5, 148.5)
- added R55: R, Resistor_SMD:R_0805_2012Metric, F.Cu at (595.2, 90.0)
- added R56: R, Resistor_SMD:R_0805_2012Metric, F.Cu at (588.1, 97.3)
- added R57: R, Resistor_SMD:R_0805_2012Metric, F.Cu at (598.6, 90.0)
- added R58: R, Resistor_SMD:R_0805_2012Metric, F.Cu at (588.1, 99.3)
- added R59: R, Resistor_SMD:R_0805_2012Metric, F.Cu at (579.1, 109.1)
- added R6: R, Resistor_SMD:R_0805_2012Metric, F.Cu at (539.5, 140.7)
- added R60: R, Resistor_SMD:R_0805_2012Metric, F.Cu at (582.6, 105.4)
- added R61: R, Resistor_SMD:R_0805_2012Metric, F.Cu at (586.2, 101.5)
- added R62: R, Resistor_SMD:R_0805_2012Metric, F.Cu at (554.3, 133.3)
- added R63: R, Resistor_SMD:R_0805_2012Metric, F.Cu at (550.9, 137.2)
- added R64: R, Resistor_SMD:R_0805_2012Metric, F.Cu at (601.6, 88.0)
- added R65: R, Resistor_SMD:R_0805_2012Metric, F.Cu at (554.3, 135.2)
- added R66: R, Resistor_SMD:R_0805_2012Metric, F.Cu at (540.9, 148.5)
- added R67: R, Resistor_SMD:R_0805_2012Metric, F.Cu at (575.7, 113.6)
- added R68: R, Resistor_SMD:R_0805_2012Metric, F.Cu at (527.3, 147.5)
- added R69: R, Resistor_SMD:R_0805_2012Metric, F.Cu at (600.1, 91.9)
- added R7: R, Resistor_SMD:R_0805_2012Metric, F.Cu at (536.1, 142.7)
- added R70: R, Resistor_SMD:R_0805_2012Metric, F.Cu at (549.7, 140.7)
- added R71: R, Resistor_SMD:R_0805_2012Metric, F.Cu at (586.2, 103.5)
- added R72: R, Resistor_SMD:R_0805_2012Metric, F.Cu at (582.6, 107.4)
- added R73: R, Resistor_SMD:R_0805_2012Metric, F.Cu at (579.1, 111.0)
- added R74: R, Resistor_SMD:R_0805_2012Metric, F.Cu at (596.7, 91.9)
- added R75: R, Resistor_SMD:R_0805_2012Metric, F.Cu at (595.0, 95.1)
- added R76: R, Resistor_SMD:R_0805_2012Metric, F.Cu at (546.3, 144.6)
- added R77: R, Resistor_SMD:R_0805_2012Metric, F.Cu at (542.9, 146.6)
- added R78: R, Resistor_SMD:R_0805_2012Metric, F.Cu at (591.6, 99.3)
- added R79: R, Resistor_SMD:R_0805_2012Metric, F.Cu at (563.1, 129.1)
- added R8: R, Resistor_SMD:R_0805_2012Metric, F.Cu at (532.7, 140.7)
- added R80: R, Resistor_SMD:R_0805_2012Metric, F.Cu at (595.0, 97.0)
- added R81: R, Resistor_SMD:R_0805_2012Metric, F.Cu at (557.7, 131.0)
- added R82: R, Resistor_SMD:R_0805_2012Metric, F.Cu at (579.1, 113.0)
- added R83: R, Resistor_SMD:R_0805_2012Metric, F.Cu at (582.6, 109.3)
- added R84: R, Resistor_SMD:R_0805_2012Metric, F.Cu at (586.0, 105.4)
- added R9: R, Resistor_SMD:R_0805_2012Metric, F.Cu at (532.7, 146.6)
- added R_trans1: R, Resistor_SMD:R_0805_2012Metric, F.Cu at (575.7, 115.5)
- added R_trans2: R, Resistor_SMD:R_0805_2012Metric, F.Cu at (554.3, 137.2)
- added R_trans3: R, Resistor_SMD:R_0805_2012Metric, F.Cu at (559.7, 129.1)
- added Transistor1: 2SC1815, Package_TO_SOT_SMD:SOT-23, F.Cu at (617.2, 51.8)
- added Transistor2: 2SC1815, Package_TO_SOT_SMD:SOT-23, F.Cu at (617.2, 55.3)
- added Transistor3: 2SC1815, Package_TO_SOT_SMD:SOT-23, F.Cu at (617.2, 58.9)
- added ext_1: ext_module_comp, sw_fprint_wLed:ext_module_footprint, F.Cu at (440.2, 120.6)
- BACKSLASH1, TAB1: footprint sw_fprint_wLed:CHERRY_PCB_100H -> sw_fprint_wLed:CHERRY_PCB_150H
- BACKSPACE1: footprint sw_fprint_wLed:CHERRY_PCB_100H -> sw_fprint_wLed:CHERRY_PCB_200H
- CAPLOCK1, RSHIFT1: footprint sw_fprint_wLed:CHERRY_PCB_100H -> sw_fprint_wLed:CHERRY_PCB_175H
- COMMAND1, LALT1, LCTRL1: footprint sw_fprint_wLed:CHERRY_PCB_100H -> sw_fprint_wLed:CHERRY_PCB_125H
- ENTER1, LSHIFT1: footprint sw_fprint_wLed:CHERRY_PCB_100H -> sw_fprint_wLed:CHERRY_PCB_225H
- SPACE1: footprint sw_fprint_wLed:CHERRY_PCB_100H -> sw_fprint_wLed:CHERRY_PCB_625H
- moved DELETE1 208.3 mm to (355.3, 77.2)
- moved HOME1 203.0 mm to (355.3, 96.3)
- moved PAGEUP1 199.4 mm to (355.3, 115.3)
- moved RIGHT1 199.3 mm to (355.3, 172.5)
- moved PAGEDOWN1 197.5 mm to (355.3, 134.4)
- moved END1 197.5 mm to (355.3, 153.4)
- moved INSERT1 190.3 mm to (336.2, 77.2)
- moved DOWN1 180.5 mm to (336.2, 172.5)
- moved UP1 178.5 mm to (336.2, 153.4)
- moved BACKSLASH1 175.8 mm to (331.5, 115.3)
- moved BACKSPACE1 175.3 mm to (326.7, 96.3)
- moved PRINTSCREEN1 172.6 mm to (317.2, 77.2)
- moved ENTER1 166.6 mm to (324.3, 134.4)
- moved LEFT1 161.7 mm to (317.2, 172.5)
- moved F12 155.2 mm to (298.1, 77.2)
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Connections:
- Aa1 pad 1: (no net) -> Net-(Aa1-Pad1)
- Aa1 pad 3: (no net) -> Net-(Aa1-Pad3)
- BACKSLASH1 pad 1: (no net) -> Net-(BACKSLASH1-Pad1)
- BACKSLASH1 pad 3: (no net) -> Net-(BACKSLASH1-Pad3)
- BACKSPACE1 pad 1: (no net) -> Net-(BACKSPACE1-Pad1)
- BACKSPACE1 pad 3: (no net) -> Net-(BACKSPACE1-Pad3)
- Bb1 pad 1: (no net) -> Net-(Bb1-Pad1)
- Bb1 pad 3: (no net) -> Net-(Bb1-Pad3)
- CAPLOCK1 pad 1: (no net) -> Net-(CAPLOCK1-Pad1)
- CAPLOCK1 pad 3: (no net) -> Net-(CAPLOCK1-Pad3)
- COMMA1 pad 1: (no net) -> Net-(COMMA1-Pad1)
- COMMA1 pad 3: (no net) -> Net-(COMMA1-Pad3)
- COMMAND1 pad 1: (no net) -> Net-(COMMAND1-Pad1)
- COMMAND1 pad 3: (no net) -> Net-(COMMAND1-Pad3)
- Cc1 pad 1: (no net) -> Net-(Cc1-Pad1)
- Cc1 pad 3: (no net) -> Net-(Cc1-Pad3)
- DELETE1 pad 1: (no net) -> Net-(D79-Pad1)
- DELETE1 pad 3: (no net) -> Net-(DELETE1-Pad3)
- DOT1 pad 1: (no net) -> Net-(D59-Pad1)
- DOT1 pad 3: (no net) -> Net-(DOT1-Pad3)
- DOWN1 pad 1: (no net) -> Net-(D78-Pad1)
- DOWN1 pad 3: (no net) -> Net-(DOWN1-Pad3)
- Dd1 pad 1: (no net) -> Net-(D22-Pad1)
- Dd1 pad 3: (no net) -> Net-(Dd1-Pad3)
- EIGHT8 pad 1: (no net) -> Net-(D39-Pad1)
- EIGHT8 pad 3: (no net) -> Net-(EIGHT8-Pad3)
- END1 pad 1: (no net) -> Net-(D83-Pad1)
- END1 pad 3: (no net) -> Net-(END1-Pad3)
- ENTER1 pad 1: (no net) -> Net-(D76-Pad1)
- ENTER1 pad 3: (no net) -> Net-(ENTER1-Pad3)
- EQUAL1 pad 1: (no net) -> Net-(D62-Pad1)
- EQUAL1 pad 3: (no net) -> Net-(EQUAL1-Pad3)
- ESC1 pad 1: (no net) -> Net-(D1-Pad1)
- ESC1 pad 3: (no net) -> Net-(ESC1-Pad3)
- Ee1 pad 1: (no net) -> Net-(D21-Pad1)
- Ee1 pad 3: (no net) -> Net-(Ee1-Pad3)
- F1 pad 1: (no net) -> Net-(D7-Pad1)
- F1 pad 3: (no net) -> Net-(F1-Pad3)
- F10 pad 1: (no net) -> Net-(D49-Pad1)
- F10 pad 3: (no net) -> Net-(F10-Pad3)
- F11 pad 1: (no net) -> Net-(D55-Pad1)
- F11 pad 3: (no net) -> Net-(F11-Pad3)
- F12 pad 1: (no net) -> Net-(D61-Pad1)
- F12 pad 3: (no net) -> Net-(F12-Pad3)
- F2 pad 1: (no net) -> Net-(D13-Pad1)
- F2 pad 3: (no net) -> Net-(F2-Pad3)
- F3 pad 1: (no net) -> Net-(D19-Pad1)
- F3 pad 3: (no net) -> Net-(F3-Pad3)
- F4 pad 1: (no net) -> Net-(D26-Pad1)
- F4 pad 3: (no net) -> Net-(F4-Pad3)
- F5 pad 1: (no net) -> Net-(D25-Pad1)
- F5 pad 3: (no net) -> Net-(F5-Pad3)
- F6 pad 1: (no net) -> Net-(D31-Pad1)
- F6 pad 3: (no net) -> Net-(F6-Pad3)
- F7 pad 1: (no net) -> Net-(D37-Pad1)
- F7 pad 3: (no net) -> Net-(F7-Pad3)
- F8 pad 1: (no net) -> Net-(D43-Pad1)
- F8 pad 3: (no net) -> Net-(F8-Pad3)
- F9 pad 1: (no net) -> Net-(D44-Pad1)
- F9 pad 3: (no net) -> Net-(F9-Pad3)
- FIVE5 pad 1: (no net) -> Net-(D33-Pad1)
- FIVE5 pad 3: (no net) -> Net-(FIVE5-Pad3)
- FOUR4 pad 1: (no net) -> Net-(D27-Pad1)
- FOUR4 pad 3: (no net) -> Net-(FOUR4-Pad3)
- FUNC1 pad 1: (no net) -> Net-(D66-Pad1)
- FUNC1 pad 3: (no net) -> Net-(FUNC1-Pad3)
- Ff1 pad 1: (no net) -> Net-(D29-Pad1)
- Ff1 pad 3: (no net) -> Net-(Ff1-Pad3)
- GRAVE1 pad 1: (no net) -> Net-(D2-Pad1)
- GRAVE1 pad 3: (no net) -> Net-(GRAVE1-Pad3)
- Gg1 pad 1: (no net) -> Net-(D36-Pad1)
- Gg1 pad 3: (no net) -> Net-(Gg1-Pad3)
- HOME1 pad 1: (no net) -> Net-(D80-Pad1)
- HOME1 pad 3: (no net) -> Net-(HOME1-Pad3)
- Hh1 pad 1: (no net) -> Net-(D41-Pad1)
- Hh1 pad 3: (no net) -> Net-(Hh1-Pad3)
- INSERT1 pad 1: (no net) -> Net-(D73-Pad1)
- INSERT1 pad 3: (no net) -> Net-(INSERT1-Pad3)
- Ii1 pad 1: (no net) -> Net-(D46-Pad1)
- Ii1 pad 3: (no net) -> Net-(Ii1-Pad3)
- Jj1 pad 1: (no net) -> Net-(D47-Pad1)
- Jj1 pad 3: (no net) -> Net-(Jj1-Pad3)
- Kk1 pad 1: (no net) -> Net-(D52-Pad1)
- Kk1 pad 3: (no net) -> Net-(Kk1-Pad3)
- LALT1 pad 1: (no net) -> Net-(D18-Pad1)
- LALT1 pad 3: (no net) -> Net-(LALT1-Pad3)
- LBRAKET1 pad 1: (no net) -> Net-(D63-Pad1)
- LBRAKET1 pad 3: (no net) -> Net-(LBRAKET1-Pad3)
- LCTRL1 pad 1: (no net) -> Net-(D6-Pad1)
- LCTRL1 pad 3: (no net) -> Net-(LCTRL1-Pad3)
- LEFT1 pad 1: (no net) -> Net-(D71-Pad1)
- LEFT1 pad 3: (no net) -> Net-(LEFT1-Pad3)
- LSHIFT1 pad 1: (no net) -> Net-(D5-Pad1)
- LSHIFT1 pad 3: (no net) -> Net-(LSHIFT1-Pad3)
- Ll1 pad 1: (no net) -> Net-(D58-Pad1)
- Ll1 pad 3: (no net) -> Net-(Ll1-Pad3)
- MINUS1 pad 1: (no net) -> Net-(D56-Pad1)
- MINUS1 pad 3: (no net) -> Net-(MINUS1-Pad3)
- Mm1 pad 1: (no net) -> Net-(D54-Pad1)
- Mm1 pad 3: (no net) -> Net-(Mm1-Pad3)
- NINE9 pad 1: (no net) -> Net-(D45-Pad1)
- NINE9 pad 3: (no net) -> Net-(NINE9-Pad3)
- Nn1 pad 1: (no net) -> Net-(D48-Pad1)
- Nn1 pad 3: (no net) -> Net-(Nn1-Pad3)
- ONE1 pad 1: (no net) -> Net-(D8-Pad1)
- ONE1 pad 3: (no net) -> Net-(ONE1-Pad3)
- Oo1 pad 1: (no net) -> Net-(D51-Pad1)
- Oo1 pad 3: (no net) -> Net-(Oo1-Pad3)
- PAGEDOWN1 pad 1: (no net) -> Net-(D82-Pad1)
- PAGEDOWN1 pad 3: (no net) -> Net-(PAGEDOWN1-Pad3)
- PAGEUP1 pad 1: (no net) -> Net-(D81-Pad1)
- PAGEUP1 pad 3: (no net) -> Net-(PAGEUP1-Pad3)
- PRINTSCREEN1 pad 1: (no net) -> Net-(D67-Pad1)
- PRINTSCREEN1 pad 3: (no net) -> Net-(PRINTSCREEN1-Pad3)
- Pp1 pad 1: (no net) -> Net-(D57-Pad1)
- Pp1 pad 3: (no net) -> Net-(Pp1-Pad3)
- QUOTE1 pad 1: (no net) -> Net-(D69-Pad1)
- QUOTE1 pad 3: (no net) -> Net-(QUOTE1-Pad3)
- Qq1 pad 1: (no net) -> Net-(D9-Pad1)
- Qq1 pad 3: (no net) -> Net-(Qq1-Pad3)
- RALT1 pad 1: (no net) -> Net-(D60-Pad1)
- RALT1 pad 3: (no net) -> Net-(R60-Pad2)
- RBRAKET1 pad 1: (no net) -> Net-(D68-Pad1)
- RBRAKET1 pad 3: (no net) -> Net-(R68-Pad2)
- RCTRL1 pad 1: (no net) -> Net-(D72-Pad1)
- RCTRL1 pad 3: (no net) -> Net-(R72-Pad2)
- RIGHT1 pad 1: (no net) -> Net-(D84-Pad1)
- RIGHT1 pad 3: (no net) -> Net-(R84-Pad2)
- RSHIFT1 pad 1: (no net) -> Net-(D70-Pad1)
- RSHIFT1 pad 3: (no net) -> Net-(R70-Pad2)
- Rr1 pad 1: (no net) -> Net-(D28-Pad1)
- Rr1 pad 3: (no net) -> Net-(R28-Pad2)
- SEMICOLON1 pad 1: (no net) -> Net-(D64-Pad1)
- SEMICOLON1 pad 3: (no net) -> Net-(R64-Pad2)
- SEVEN7 pad 1: (no net) -> Net-(D38-Pad1)
- SEVEN7 pad 3: (no net) -> Net-(R38-Pad2)
- SIX6 pad 1: (no net) -> Net-(D32-Pad1)
- SIX6 pad 3: (no net) -> Net-(R32-Pad2)
- SLASH1 pad 1: (no net) -> Net-(D65-Pad1)
- SLASH1 pad 3: (no net) -> Net-(R65-Pad2)
- SPACE1 pad 1: (no net) -> Net-(D24-Pad1)
- SPACE1 pad 3: (no net) -> Net-(R24-Pad2)
- Ss1 pad 1: (no net) -> Net-(D16-Pad1)
- Ss1 pad 3: (no net) -> Net-(R16-Pad2)
- TAB1 pad 1: (no net) -> Net-(D3-Pad1)
- TAB1 pad 3: (no net) -> Net-(R3-Pad2)
- THREE3 pad 1: (no net) -> Net-(D20-Pad1)
- THREE3 pad 3: (no net) -> Net-(R20-Pad2)
- TWO2 pad 1: (no net) -> Net-(D14-Pad1)
- TWO2 pad 3: (no net) -> Net-(R14-Pad2)
- Tt1 pad 1: (no net) -> Net-(D34-Pad1)
- Tt1 pad 3: (no net) -> Net-(R34-Pad2)
- UP1 pad 1: (no net) -> Net-(D77-Pad1)
- UP1 pad 3: (no net) -> Net-(R77-Pad2)
- Uu1 pad 1: (no net) -> Net-(D40-Pad1)
- Uu1 pad 3: (no net) -> Net-(R40-Pad2)
- Vv1 pad 1: (no net) -> Net-(D30-Pad1)
- Vv1 pad 3: (no net) -> Net-(R30-Pad2)
- Ww1 pad 1: (no net) -> Net-(D15-Pad1)
- Ww1 pad 3: (no net) -> Net-(R15-Pad2)
- Xx1 pad 1: (no net) -> Net-(D17-Pad1)
- Xx1 pad 3: (no net) -> Net-(R17-Pad2)
- Yy1 pad 1: (no net) -> Net-(D35-Pad1)
- Yy1 pad 3: (no net) -> Net-(R35-Pad2)
- ZERO0 pad 1: (no net) -> Net-(D50-Pad1)
- ZERO0 pad 3: (no net) -> Net-(R50-Pad2)
- Zz1 pad 1: (no net) -> Net-(D11-Pad1)
- Zz1 pad 3: (no net) -> Net-(R11-Pad2)

Commit message: diode placement
Parts:
- D1, D10, D11, D12, D13, D14, D15, D16, D17, D18, D19, D2, D20, D21, D22, D23, D24, D25, D26, D27, D28, D29, D3, D30, D31, D32, D33, D34, D35, D36, D37, D38, D39, D4, D40, D41, D42, D43, D44, D45, D46, D47, D48, D49, D5, D50, D51, D52, D53, D54, D55, D56, D57, D58, D59, D6, D60, D61, D62, D63, D64, D65, D66, D67, D68, D69, D7, D70, D71, D72, D73, D74, D75, D76, D77, D78, D79, D8, D80, D81, D82, D83, D84, D9: footprint Diode_SMD:D_MiniMELF -> sw_fprint_wLed:D_MiniMELFr
- MCU1: footprint sw_fprint_wLed:Teensy2.0++_footprint_assigned -> sw_fprint_wLed:Teensy2.0++_footprint
- R1, R10, R11, R12, R13, R14, R15, R16, R17, R18, R19, R2, R20, R21, R22, R23, R24, R25, R26, R27, R28, R29, R3, R30, R31, R32, R33, R34, R35, R36, R37, R38, R39, R4, R40, R41, R42, R43, R44, R45, R46, R47, R48, R49, R5, R50, R51, R52, R53, R54, R55, R56, R57, R58, R59, R6, R60, R61, R62, R63, R64, R65, R66, R67, R68, R69, R7, R70, R71, R72, R73, R74, R75, R76, R77, R78, R79, R8, R80, R81, R82, R83, R84, R9: moved to B.Cu
- moved D9 527.7 mm to (89.8, 122.2), turned to 270 degrees
- moved D11 466.8 mm to (103.8, 160.3), turned to 270 degrees
- moved D23 434.7 mm to (141.9, 160.3), turned to 270 degrees
- moved D3 424.6 mm to (61.3, 122.2), turned to 270 degrees
- moved R11 414.5 mm to (252.9, 263.1)
- moved R5 411.0 mm to (252.6, 259.5)
- moved R3 411.0 mm to (249.2, 259.5)
- moved D18 410.3 mm to (108.9, 179.3), turned to 270 degrees
- moved D20 401.6 mm to (118.4, 103.1), turned to 270 degrees
- moved D21 395.8 mm to (127.9, 122.2), turned to 270 degrees
- moved D6 393.9 mm to (61.3, 179.3), turned to 270 degrees
- moved D14 393.2 mm to (99.4, 103.1), turned to 270 degrees
- moved D1 391.0 mm to (61.3, 84.1), turned to 270 degrees
- moved D17 389.6 mm to (122.9, 160.3), turned to 270 degrees
- moved D2 383.6 mm to (61.3, 103.1), turned to 270 degrees
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
Commit message: update pcb
Parts:
- MCU1: footprint sw_fprint_wLed:Teensy2.0++_footprint -> sw_fprint_wLed:Teensy2.0++_footprint_assigned

Commit message: update
Parts:
- moved ext_1 275.7 mm to (165.4, 99.1)
- moved MCU1 120.2 mm to (89.8, 67.5), turned to 0 degrees
- moved R82 48.5 mm to (212.7, 197.9)
- moved D1 3.17 mm to (64.4, 84.1)
- moved D2 3.17 mm to (64.4, 103.1)
Other:
- outline, holes or cut-outs redrawn

Commit message: almost
Parts:
- R_trans1, R_trans2, R_trans3, Transistor1, Transistor2, Transistor3: moved to B.Cu
- moved P_jump_trans1 368.6 mm to (58.7, 56.3)
- moved P_jump_trans2 365.7 mm to (58.7, 51.2)
- moved P_jump_trans3 363.7 mm to (58.7, 53.7)
- moved Transistor2 351.3 mm to (63.5, 51.6), turned to 270 degrees
- moved Transistor3 351.2 mm to (63.5, 55.8), turned to 270 degrees
- moved Transistor1 347.7 mm to (63.5, 59.6), turned to 270 degrees
- moved R_trans2 342.1 mm to (71.7, 53.0), turned to 180 degrees
- moved R_trans1 336.9 mm to (71.7, 61.2)
- moved R_trans3 335.7 mm to (71.7, 56.8)
- moved R1 242.2 mm to (65.1, 72.1)
- moved R13 240.0 mm to (103.2, 72.1)
- moved R7 234.4 mm to (83.5, 72.1)
- moved R3 233.8 mm to (69.2, 110.2)
- moved R2 233.5 mm to (64.4, 91.2)
- moved R19 230.9 mm to (121.6, 72.1)
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Routing:
- net Net-(BACKSPACE1-Pad4): track 0.00 -> 650.8 mm
- net Net-(D12-Pad2): track 0.00 -> 394.4 mm
- net Net-(D11-Pad2): track 0.00 -> 384.5 mm
- net Net-(D10-Pad2): track 0.00 -> 378.1 mm
- net Net-(D14-Pad2): track 0.00 -> 365.4 mm
- net Net-(D15-Pad2): track 0.00 -> 347.2 mm
- net Net-(D1-Pad2): track 0.00 -> 325.1 mm
- net Net-(LEFT1-Pad2): track 0.00 -> 139.1 mm
- net Net-(Cc1-Pad2): track 0.00 -> 135.4 mm
- net Net-(BACKSLASH1-Pad2): track 0.00 -> 114.0 mm
- net Net-(Aa1-Pad2): track 0.00 -> 112.1 mm
- net Net-(DOT1-Pad2): track 0.00 -> 111.0 mm
- net Net-(EQUAL1-Pad2): track 0.00 -> 111.0 mm
- net Net-(F2-Pad2): track 0.00 -> 110.0 mm
- net Net-(Bb1-Pad2): track 0.00 -> 110.0 mm
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
Commit message: update led1
Parts:
- R_trans1, R_trans2, R_trans3, Transistor1, Transistor2, Transistor3: moved to F.Cu
- moved R_trans3 6.81 mm to (68.9, 50.6)
- moved Transistor3 5.14 mm to (63.6, 50.7), turned to 0 degrees
- moved P_jump_trans2 4.02 mm to (57.5, 55.0)
- moved R_trans1 4.01 mm to (69.0, 58.3)
- moved R_trans2 3.13 mm to (68.9, 54.5), turned to 0 degrees
- moved Transistor2 2.91 mm to (63.5, 54.6), turned to 0 degrees
- moved P_jump_trans1 1.80 mm to (57.5, 57.5)
- moved P_jump_trans3 1.80 mm to (57.5, 52.5)
- moved Transistor1 1.27 mm to (63.5, 58.4), turned to 0 degrees
- moved R83 0.90 mm to (350.5, 148.3)
- moved R47 0.76 mm to (212.2, 129.3)
- moved R35 0.73 mm to (188.5, 110.2)
- moved R18 0.56 mm to (114.7, 167.4)
- moved R77 0.51 mm to (331.4, 148.3)
- moved R84 0.51 mm to (350.4, 167.4)
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Routing:
- net Net-(BACKSPACE1-Pad4): track 650.8 -> 1273.2 mm
- net Net-(MCU1-Pad26): track 0.00 -> 32.4 mm
- net Net-(MCU1-Pad25): track 0.00 -> 31.9 mm
- net Net-(MCU1-Pad24): track 0.00 -> 31.2 mm
- net Net-(MCU1-Pad51): track 0.00 -> 13.6 mm
- net Net-(Aa1-Pad4): track 0.00 -> 6.00 mm
- net Net-(Bb1-Pad4): track 0.00 -> 5.81 mm
- net Net-(R_trans1-Pad1): track 0.00 -> 3.52 mm
- net Net-(DOT1-Pad3): track 0.00 -> 3.49 mm
- net Net-(R_trans2-Pad1): track 0.00 -> 3.49 mm
- net Net-(R_trans3-Pad1): track 0.00 -> 3.48 mm
- net Net-(R34-Pad2): track 0.00 -> 3.18 mm
- net Net-(PAGEUP1-Pad3): track 0.00 -> 3.18 mm
- net Net-(R28-Pad2): track 0.00 -> 3.17 mm
- net Net-(R3-Pad2): track 0.00 -> 2.89 mm
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- added copper zone on B.Cu, net Net-(MCU1-Pad46)
- added copper zone on F.Cu, net Net-(MCU1-Pad49)

Commit message: update pinout, flip teensy
Parts:
- MCU1: moved to B.Cu
- moved MCU1 17.4 mm to (89.8, 50.3)
Connections:
- MCU1 pad 18: Net-(COMMA1-Pad2) -> Net-(F6-Pad2)
- MCU1 pad 19: Net-(DOT1-Pad2) -> Net-(F4-Pad2)
- MCU1 pad 2: Net-(CAPLOCK1-Pad2) -> Net-(F8-Pad2)
- MCU1 pad 20: Net-(EQUAL1-Pad2) -> Net-(Cc1-Pad2)
- MCU1 pad 21: Net-(LEFT1-Pad2) -> Net-(F2-Pad2)
- MCU1 pad 22: Net-(BACKSLASH1-Pad2) -> Net-(Aa1-Pad2)
- MCU1 pad 23: Net-(DELETE1-Pad2) -> Net-(CAPLOCK1-Pad2)
- MCU1 pad 3: Net-(Aa1-Pad2) -> Net-(COMMA1-Pad2)
- MCU1 pad 38: Net-(F8-Pad2) -> Net-(Bb1-Pad2)
- MCU1 pad 4: Net-(F2-Pad2) -> Net-(DOT1-Pad2)
- MCU1 pad 5: Net-(Cc1-Pad2) -> Net-(EQUAL1-Pad2)
- MCU1 pad 51: Net-(MCU1-Pad51) -> (no net)
- MCU1 pad 52: Net-(MCU1-Pad52) -> (no net)
- MCU1 pad 6: Net-(F4-Pad2) -> Net-(LEFT1-Pad2)
- MCU1 pad 7: Net-(F6-Pad2) -> Net-(BACKSLASH1-Pad2)
- MCU1 pad 8: Net-(Bb1-Pad2) -> Net-(DELETE1-Pad2)
- ext_1 pad 2: Net-(ext_1-Pad2) -> (no net)
- ext_1 pad 3: Net-(ext_1-Pad3) -> (no net)
Routing:
- net Net-(Bb1-Pad4): track 5.81 -> 1150.2 mm
- net Net-(Aa1-Pad4): track 6.00 -> 825.7 mm
- net Net-(D15-Pad2): track 347.2 -> 481.0 mm
- net Net-(D14-Pad2): track 365.4 -> 475.8 mm
- net Net-(Bb1-Pad2): track 110.0 -> 211.9 mm
- net Net-(BACKSPACE1-Pad4): track 1273.2 -> 1182.1 mm
- net Net-(F6-Pad2): track 101.2 -> 186.2 mm
- net Net-(D1-Pad2): track 325.1 -> 387.1 mm
- net Net-(F4-Pad2): track 107.0 -> 156.1 mm
- net Net-(Cc1-Pad2): track 135.4 -> 177.3 mm
- net Net-(CAPLOCK1-Pad2): track 104.1 -> 144.9 mm
- net Net-(EQUAL1-Pad2): track 111.0 -> 138.5 mm
- net Net-(Aa1-Pad2): track 112.1 -> 133.3 mm
- net Net-(F2-Pad2): track 110.0 -> 131.1 mm
- net Net-(MCU1-Pad51): track 13.6 -> 0.00 mm
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