File: main_board4.sch (KiCad schematic (older format))
At the start: 288 parts

Commit message: big chang
Parts:
- removed 5volt1, Ground1, P_control_led1, P_control_led2, P_control_led3, col1, col10, col11, col12, col13, col14, col2, col3, col4, col5, col6, col7, col8, col9, row1, row2, row3, row4, row5, row6: CONN_01X01, Connector_PinHeader_2.54mm:PinHeader_1x01_P2.54mm_Vertical, symbol lee_mech_key_comp:CONN_01X01
Connections:
- net at CAPLOCK1.2, ESC1.2, GRAVE1.2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: now also CAPLOCK1.3 (led+), ESC1.3 (led+), GRAVE1.3 (led+), LSHIFT1.3 (led+), MCU1.2 (D2), R1.2, R2.2, R3.2, R4.2, R5.2, TAB1.3 (led+)
- net at Aa1.2, COMMAND1.2, F1.2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: now also Aa1.3 (led+), F1.3 (led+), MCU1.3 (D3), ONE1.3 (led+), Qq1.3 (led+), R10.2, R11.2, R7.2, R8.2, R9.2, Zz1.3 (led+)
- net at F2.2, LALT1.2, Ss1.2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: now also F2.3 (led+), MCU1.4 (D4), R13.2, R14.2, R15.2, R16.2, R17.2, Ss1.3 (led+), TWO2.3 (led+), Ww1.3 (led+), Xx1.3 (led+)
- net at Cc1.2, Dd1.2, Ee1.2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: now also Cc1.3 (led+), Dd1.3 (led+), Ee1.3 (led+), F3.3 (led+), MCU1.5 (D5), R19.2, R20.2, R21.2, R22.2, R23.2, THREE3.3 (led+)
- net at F4.2, F5.2, FOUR4.2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: now also F4.3 (led+), F5.3 (led+), FOUR4.3 (led+), Ff1.3 (led+), MCU1.6 (D6), R25.2, R26.2, R27.2, R28.2, R29.2, Rr1.3 (led+)
- net at F6.2, FIVE5.2, Gg1.2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: now also F6.3 (led+), FIVE5.3 (led+), MCU1.7 (D7), R31.2, R32.2, R33.2, R34.2, R35.2, SIX6.3 (led+), Tt1.3 (led+), Yy1.3 (led+)
- net at Bb1.2, EIGHT8.2, F7.2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: now also EIGHT8.3 (led+), F7.3 (led+), Hh1.3 (led+), MCU1.8 (E0), R37.2, R38.2, R39.2, R40.2, R41.2, SEVEN7.3 (led+), Uu1.3 (led+)
- net at F8.2, F9.2, Ii1.2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: now also F8.3 (led+), F9.3 (led+), Ii1.3 (led+), Jj1.3 (led+), MCU1.38 (F0), NINE9.3 (led+), R43.2, R44.2, R45.2, R46.2, R47.2
- net at COMMA1.2, F10.2, Kk1.2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: now also COMMA1.3 (led+), F10.3 (led+), Kk1.3 (led+), MCU1.18 (E6), Oo1.3 (led+), R49.2, R50.2, R51.2, R52.2, R53.2, ZERO0.3 (led+)
- net at DOT1.2, F11.2, Ll1.2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: now also DOT1.3 (led+), F11.3 (led+), Ll1.3 (led+), MCU1.19 (E7), MINUS1.3 (led+), Pp1.3 (led+), R55.2, R56.2, R57.2, R58.2, R59.2
- net at EQUAL1.2, F12.2, FUNC1.2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: now also EQUAL1.3 (led+), F12.3 (led+), LBRAKET1.3 (led+), MCU1.20 (B0), R61.2, R62.2, R63.2, R64.2, R65.2, SEMICOLON1.3 (led+), SLASH1.3 (led+)
- net at LEFT1.2, PRINTSCREEN1.2, QUOTE1.2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: now also LEFT1.3 (led+), MCU1.21 (B1), PRINTSCREEN1.3 (led+), QUOTE1.3 (led+), R67.2, R68.2, R69.2, R70.2, R71.2, RBRAKET1.3 (led+), RSHIFT1.3 (led+)
- net at BACKSLASH1.2, BACKSPACE1.2, DOWN1.2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: now also BACKSLASH1.3 (led+), BACKSPACE1.3 (led+), ENTER1.3 (led+), INSERT1.3 (led+), MCU1.22 (B2), R73.2, R74.2, R75.2, R76.2, R77.2, UP1.3 (led+)
- net at DELETE1.2, END1.2, HOME1.2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: now also DELETE1.3 (led+), END1.3 (led+), HOME1.3 (led+), MCU1.23 (B3), PAGEDOWN1.3 (led+), PAGEUP1.3 (led+), R79.2, R80.2, R81.2, R82.2, R83.2
- net at D11.2 (K), D17.2 (K), D23.2 (K)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: now also MCU1.41 (F3)
- net at D12.2 (K), D18.2 (K), D24.2 (K)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: now also MCU1.40 (F2)
- net at D10.2 (K), D16.2 (K), D22.2 (K)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: now also MCU1.42 (F4)
- net at D15.2 (K), D21.2 (K), D27.2 (K)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: now also MCU1.14 (C4)
- net at D14.2 (K), D2.2 (K), D20.2 (K)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: now also MCU1.13 (C3)
- net at D1.2 (K), D13.2 (K), D19.2 (K)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: now also MCU1.12 (C2)
- net at Transistor1.1 (E), Transistor2.1 (E), Transistor3.1 (E): now also MCU1.49 (GND)
- net at R1.1, R10.1, R11.1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: now also MCU1.46 (5V)
- net at ext_1.5 (SCL): now also MCU1.0 (D0)
- net at ext_1.6 (SDA): now also MCU1.1 (D1)
- net at ext_1.7 (Led_control): now also MCU1.39 (F1)
- net at ext_1.8 (USB_drive_control): now also MCU1.27 (B7)
- net at MCU1.24 (B4): now also R_trans3.2
- net at MCU1.25 (B5): now also R_trans2.2
- net at MCU1.26 (B6): now also R_trans1.2
Other:
- moved on the sheet: Aa1, BACKSLASH1, BACKSPACE1, Bb1, CAPLOCK1, COMMA1, COMMAND1, Cc1, D1, D10, D11, D12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

Commit message: update
Connections:
- net at MCU1.49 (GND), Transistor1.1 (E), Transistor2.1 (E)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: now also ext_1.4 (Gnd)
- net at MCU1.46 (5V), R1.1, R10.1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: now also ext_1.1 (Vcc)
- no-connect marks 0 -> 27
Changed lines of the file:
@@
 	4250 12950 4250 9200
 Wire Wire Line
-	4250 12950 7800 12950
+	4250 12950 5600 12950
 Connection ~ 4250 9200
 Wire Wire Line
@@
 Wire Wire Line
 	9850 11200 11500 11200
+Wire Wire Line
+	5600 13350 5600 12950
+Connection ~ 5600 12950
+Wire Wire Line
+	5600 12950 7800 12950
+Wire Wire Line
+	5900 12400 7500 12400
+Wire Wire Line
+	5900 12400 5900 13350
+Connection ~ 7500 12400
+NoConn ~ 5700 13350
+NoConn ~ 5800 13350
+NoConn ~ 8300 13350
+NoConn ~ 8350 13350
+NoConn ~ 8650 13350
+NoConn ~ 8700 13350
+NoConn ~ 8750 13350
+NoConn ~ 8950 13350
+NoConn ~ 9000 13350
+NoConn ~ 9050 13350
+NoConn ~ 9100 13350
+NoConn ~ 9200 13350
+NoConn ~ 9800 13750
+NoConn ~ 9800 13900
+NoConn ~ 9800 14050
+NoConn ~ 9400 14450
+NoConn ~ 9200 14450
+NoConn ~ 9100 14450
+NoConn ~ 9050 14450
+NoConn ~ 9000 14450
+NoConn ~ 8950 14450
+NoConn ~ 8750 14450
+NoConn ~ 8700 14450
+NoConn ~ 8650 14450
+NoConn ~ 8450 14450
+NoConn ~ 8400 14450
+NoConn ~ 8350 14450
 $EndSCHEMATC

Commit message: working on pcb layout
Connections:
- new net: CAPLOCK1.2, ESC1.2, GRAVE1.2, LCTRL1.2, LSHIFT1.2, MCU1.2 (D2), TAB1.2
- new net: GRAVE1.3 (led+), R2.2
- new net: R3.2, TAB1.3 (led+)
- new net: CAPLOCK1.3 (led+), R4.2
- new net: LSHIFT1.3 (led+), R5.2
- new net: ESC1.3 (led+), R1.2
- new net: COMMA1.2, F10.2, Kk1.2, MCU1.18 (E6), Mm1.2, Oo1.2, ZERO0.2
- new net: DOT1.2, F11.2, Ll1.2, MCU1.19 (E7), MINUS1.2, Pp1.2, RALT1.2
- new net: EQUAL1.2, F12.2, FUNC1.2, LBRAKET1.2, MCU1.20 (B0), SEMICOLON1.2, SLASH1.2
- new net: LEFT1.2, MCU1.21 (B1), PRINTSCREEN1.2, QUOTE1.2, RBRAKET1.2, RCTRL1.2, RSHIFT1.2
- new net: BACKSLASH1.2, BACKSPACE1.2, DOWN1.2, ENTER1.2, INSERT1.2, MCU1.22 (B2), UP1.2
- new net: DELETE1.2, END1.2, HOME1.2, MCU1.23 (B3), PAGEDOWN1.2, PAGEUP1.2, RIGHT1.2
- new net: Aa1.2, COMMAND1.2, F1.2, MCU1.3 (D3), ONE1.2, Qq1.2, Zz1.2
- new net: F8.2, F9.2, Ii1.2, Jj1.2, MCU1.38 (F0), NINE9.2, Nn1.2
- new net: F2.2, LALT1.2, MCU1.4 (D4), Ss1.2, TWO2.2, Ww1.2, Xx1.2
- new net: Cc1.2, Dd1.2, Ee1.2, F3.2, MCU1.5 (D5), SPACE1.2, THREE3.2
- new net: F4.2, F5.2, FOUR4.2, Ff1.2, MCU1.6 (D6), Rr1.2, Vv1.2
- new net: F6.2, FIVE5.2, Gg1.2, MCU1.7 (D7), SIX6.2, Tt1.2, Yy1.2
- new net: Bb1.2, EIGHT8.2, F7.2, Hh1.2, MCU1.8 (E0), SEVEN7.2, Uu1.2
- new net: F1.3 (led+), R7.2
- new net: ONE1.3 (led+), R8.2
- new net: Qq1.3 (led+), R9.2
- new net: Aa1.3 (led+), R10.2
- new net: R11.2, Zz1.3 (led+)
- new net: F2.3 (led+), R13.2
- new net: R14.2, TWO2.3 (led+)
- new net: R15.2, Ww1.3 (led+)
- new net: R16.2, Ss1.3 (led+)
- new net: R17.2, Xx1.3 (led+)
- new net: F3.3 (led+), R19.2
- new net: R20.2, THREE3.3 (led+)
- new net: Ee1.3 (led+), R21.2
- new net: Dd1.3 (led+), R22.2
- new net: Cc1.3 (led+), R23.2
- new net: F5.3 (led+), R25.2
- new net: F4.3 (led+), R26.2
- new net: FOUR4.3 (led+), R27.2
- new net: R28.2, Rr1.3 (led+)
- new net: Ff1.3 (led+), R29.2
- new net: F6.3 (led+), R31.2
- new net: R32.2, SIX6.3 (led+)
- new net: FIVE5.3 (led+), R33.2
- new net: R34.2, Tt1.3 (led+)
- new net: R35.2, Yy1.3 (led+)
- new net: F7.3 (led+), R37.2
- new net: R38.2, SEVEN7.3 (led+)
- new net: EIGHT8.3 (led+), R39.2
- new net: R40.2, Uu1.3 (led+)
- new net: Hh1.3 (led+), R41.2
- new net: F8.3 (led+), R43.2
- new net: F9.3 (led+), R44.2
- new net: NINE9.3 (led+), R45.2
- new net: Ii1.3 (led+), R46.2
- new net: Jj1.3 (led+), R47.2
- new net: F10.3 (led+), R49.2
- new net: R50.2, ZERO0.3 (led+)
- new net: Oo1.3 (led+), R51.2
- new net: Kk1.3 (led+), R52.2
- new net: COMMA1.3 (led+), R53.2
- new net: F11.3 (led+), R55.2
- new net: MINUS1.3 (led+), R56.2
- new net: Pp1.3 (led+), R57.2
- new net: Ll1.3 (led+), R58.2
- new net: DOT1.3 (led+), R59.2
- new net: F12.3 (led+), R61.2
- new net: EQUAL1.3 (led+), R62.2
- new net: LBRAKET1.3 (led+), R63.2
- new net: R64.2, SEMICOLON1.3 (led+)
- new net: R65.2, SLASH1.3 (led+)
- new net: PRINTSCREEN1.3 (led+), R67.2
- new net: R68.2, RBRAKET1.3 (led+)
- new net: QUOTE1.3 (led+), R69.2
- new net: R70.2, RSHIFT1.3 (led+)
- new net: LEFT1.3 (led+), R71.2
- new net: INSERT1.3 (led+), R73.2
- new net: BACKSPACE1.3 (led+), R74.2
- new net: BACKSLASH1.3 (led+), R75.2
- new net: ENTER1.3 (led+), R76.2
- new net: R77.2, UP1.3 (led+)
- new net: DELETE1.3 (led+), R79.2
- new net: HOME1.3 (led+), R80.2
- new net: PAGEUP1.3 (led+), R81.2
- new net: PAGEDOWN1.3 (led+), R82.2
- new net: END1.3 (led+), R83.2

Commit message: update pcb
Parts:
- MCU1: footprint sw_fprint_wLed:Teensy2.0++_footprint -> sw_fprint_wLed:Teensy2.0++_footprint_assigned
Connections:
- net at CAPLOCK1.2, ESC1.2, GRAVE1.2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: now also MCU1.23 (B3); no longer MCU1.2 (D2)
- net at COMMA1.2, F10.2, Kk1.2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: now also MCU1.7 (D7); no longer MCU1.18 (E6)
- net at DOT1.2, F11.2, Ll1.2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: now also MCU1.6 (D6); no longer MCU1.19 (E7)
- net at EQUAL1.2, F12.2, FUNC1.2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: now also MCU1.5 (D5); no longer MCU1.20 (B0)
- net at LEFT1.2, PRINTSCREEN1.2, QUOTE1.2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: now also MCU1.4 (D4); no longer MCU1.21 (B1)
- net at BACKSLASH1.2, BACKSPACE1.2, DOWN1.2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: now also MCU1.3 (D3); no longer MCU1.22 (B2)
- net at DELETE1.2, END1.2, HOME1.2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: now also MCU1.2 (D2); no longer MCU1.23 (B3)
- net at Aa1.2, COMMAND1.2, F1.2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: now also MCU1.22 (B2); no longer MCU1.3 (D3)
- net at F8.2, F9.2, Ii1.2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: now also MCU1.8 (E0); no longer MCU1.38 (F0)
- net at F2.2, LALT1.2, Ss1.2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: now also MCU1.21 (B1); no longer MCU1.4 (D4)
- net at Cc1.2, Dd1.2, Ee1.2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: now also MCU1.20 (B0); no longer MCU1.5 (D5)
- net at F4.2, F5.2, FOUR4.2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: now also MCU1.19 (E7); no longer MCU1.6 (D6)
- net at F6.2, FIVE5.2, Gg1.2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: now also MCU1.18 (E6); no longer MCU1.7 (D7)
- net at Bb1.2, EIGHT8.2, F7.2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: now also MCU1.38 (F0); no longer MCU1.8 (E0)
Changed lines of the file:
@@
 EESchema Schematic File Version 4
 LIBS:power
-LIBS:device
 LIBS:74xx
-LIBS:audio
-LIBS:interface
 LIBS:main_board4-cache
 EELAYER 26 0
@@
 F 0 "MCU1" H 7600 14200 60  0000 C CNN
 F 1 "Teensy2.0++" H 7750 14100 60  0000 C CNN
-F 2 "sw_fprint_wLed:Teensy2.0++_footprint" H 7750 14250 60  0001 C CNN
+F 2 "sw_fprint_wLed:Teensy2.0++_footprint_assigned" H 7750 14250 60  0001 C CNN
 F 3 "" H 7750 14250 60  0001 C CNN
 	1    7750 14250
@@
 	18400 6700 22850 6700
 Wire Wire Line
-	4200 6050 4200 14850
-Wire Wire Line
-	4200 14850 8000 14850
-Wire Wire Line
-	8000 14850 8000 14450
-Wire Wire Line
-	8050 14450 8050 14900
-Wire Wire Line
-	8050 14900 4150 14900
-Wire Wire Line
-	4150 14900 4150 6000
-Wire Wire Line
-	4100 5950 4100 14950
-Wire Wire Line
-	4100 14950 8100 14950
-Wire Wire Line
-	8100 14950 8100 14450
-Wire Wire Line
-	8150 14450 8150 15000
-Wire Wire Line
-	8150 15000 4050 15000
-Wire Wire Line
-	4050 15000 4050 5900
-Wire Wire Line
-	4000 5850 4000 15050
-Wire Wire Line
-	4000 15050 8200 15050
-Wire Wire Line
-	8200 15050 8200 14450
-Wire Wire Line
-	8250 14450 8250 15100
-Wire Wire Line
-	8250 15100 3950 15100
-Wire Wire Line
-	3950 15100 3950 5800
-Wire Wire Line
-	3800 5750 3800 15150
-Wire Wire Line
-	3800 15150 8300 15150
-Wire Wire Line
-	8300 15150 8300 14450
-Wire Wire Line
-	8400 13350 8400 13050
-Wire Wire Line
-	8400 13050 22400 13050
-Wire Wire Line
-	22400 13050 22400 5700
+	3800 5750 3800 9900
 Wire Wire Line
 	12550 5700 22400 5700
@@
 	13900 5650 22350 5650
 Wire Wire Line
-	22350 5650 22350 13000
-Wire Wire Line
-	22350 13000 8250 13000
-Wire Wire Line
-	8250 13000 8250 13350
-Wire Wire Line
-	8200 13350 8200 12950
-Wire Wire Line
-	8200 12950 22300 12950
-Wire Wire Line
-	22300 12950 22300 5600
-Wire Wire Line
 	14950 5600 22300 5600
 Wire Wire Line
-	8150 13350 8150 12900
-Wire Wire Line
-	8150 12900 22250 12900
-Wire Wire Line
-	22250 12900 22250 5550
-Wire Wire Line
 	16000 5550 22250 5550
 Wire Wire Line
-	22200 5500 22200 12850
-Wire Wire Line
-	22200 12850 8100 12850
-Wire Wire Line
-	8100 12850 8100 13350
-Wire Wire Line
-	8050 13350 8050 12800
-Wire Wire Line
-	8050 12800 22150 12800
-Wire Wire Line
-	22150 12800 22150 5450
-Wire Wire Line
 	18100 5450 22150 5450
 Wire Wire Line
@@
 	19150 5400 22100 5400
 Wire Wire Line
-	22100 5400 22100 12750
-Wire Wire Line
-	22100 12750 8000 12750
-Wire Wire Line
-	8000 12750 8000 13350
-Wire Wire Line
 	3800 5750 11500 5750
 Wire Wire Line
@@
 	4150 6000 6250 6000
 Wire Wire Line
-	4250 12950 4250 9200
-Wire Wire Line
 	4250 12950 5600 12950
 Connection ~ 4250 9200
@@
 Wire Wire Line
 	19150 6300 19150 6900
+Wire Wire Line
+	4250 9200 4250 12950
+Wire Wire Line
+	8400 9900 3800 9900
+Wire Wire Line
+	4200 6050 4200 10200
+Wire Wire Line
+	4150 6000 4150 10150
+Wire Wire Line
+	4100 5950 4100 10100
+Wire Wire Line
+	4050 5900 4050 10050
+Wire Wire Line
+	4000 5850 4000 10000
+Wire Wire Line
+	3950 5800 3950 9950
+Wire Wire Line
+	8400 9900 8400 13350
+Wire Wire Line
+	3950 9950 8250 9950
+Wire Wire Line
+	8250 9950 8250 13350
+Wire Wire Line
+	8200 10000 4000 10000
+Wire Wire Line
+	8200 10000 8200 13350
+Wire Wire Line
+	4050 10050 8150 10050
+Wire Wire Line
+	8150 10050 8150 13350
+Wire Wire Line
+	8100 10100 4100 10100
+Wire Wire Line
+	8100 10100 8100 13350
+Wire Wire Line
+	4150 10150 8050 10150
+Wire Wire Line
+	8050 10150 8050 13350
+Wire Wire Line
+	8000 10200 4200 10200
+Wire Wire Line
+	8000 10200 8000 13350
+Wire Wire Line
+	8000 15700 22100 15700
+Wire Wire Line
+	8000 14450 8000 15700
+Wire Wire Line
+	22100 5400 22100 15700
+Wire Wire Line
+	22150 15650 8050 15650
+Wire Wire Line
+	8050 14450 8050 15650
+Wire Wire Line
+	22150 5450 22150 15650
+Wire Wire Line
+	8100 15600 22200 15600
+Wire Wire Line
+	8100 14450 8100 15600
+Wire Wire Line
+	22200 5500 22200 15600
+Wire Wire Line
+	22250 15550 8150 15550
+Wire Wire Line
+	8150 14450 8150 15550
+Wire Wire Line
+	22250 5550 22250 15550
+Wire Wire Line
+	8200 15500 22300 15500
+Wire Wire Line
+	8200 14450 8200 15500
+Wire Wire Line
+	22300 5600 22300 15500
+Wire Wire Line
+	22350 15450 8250 15450
+Wire Wire Line
+	8250 14450 8250 15450
+Wire Wire Line
+	22350 5650 22350 15450
+Wire Wire Line
+	22400 15400 8300 15400
+Wire Wire Line
+	22400 5700 22400 15400
+Wire Wire Line
+	8300 14450 8300 15400
 $EndSCHEMATC

Commit message: update pinout, flip teensy
Connections:
- net at DELETE1.2, END1.2, HOME1.2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: now also MCU1.8 (E0); no longer MCU1.2 (D2)
- net at BACKSLASH1.2, BACKSPACE1.2, DOWN1.2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: now also MCU1.7 (D7); no longer MCU1.3 (D3)
- net at LEFT1.2, PRINTSCREEN1.2, QUOTE1.2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: now also MCU1.6 (D6); no longer MCU1.4 (D4)
- net at DOT1.2, F11.2, Ll1.2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: now also MCU1.4 (D4); no longer MCU1.6 (D6)
- net at COMMA1.2, F10.2, Kk1.2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: now also MCU1.3 (D3); no longer MCU1.7 (D7)
- net at F8.2, F9.2, Ii1.2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: now also MCU1.2 (D2); no longer MCU1.8 (E0)
Changed lines of the file:
@@
 EESchema Schematic File Version 4
 LIBS:power
+LIBS:device
 LIBS:74xx
+LIBS:audio
+LIBS:interface
 LIBS:main_board4-cache
 EELAYER 26 0
@@
 	17350 7300 16300 7300
 Wire Wire Line
-	19150 5400 19150 6300
+	19150 5700 19150 6300
 Wire Wire Line
-	18100 5450 18100 6300
+	18100 5650 18100 6300
 Wire Wire Line
-	17050 5500 17050 6300
+	17050 5600 17050 6300
 Wire Wire Line
 	16000 5550 16000 6300
 Wire Wire Line
-	14950 5600 14950 6300
+	14950 5450 14950 6300
 Wire Wire Line
-	13900 5650 13900 6300
+	13900 5400 13900 6300
 Wire Wire Line
-	12550 5700 12550 6300
+	12550 5350 12550 6300
 Wire Wire Line
 	11500 5750 11500 6300
@@
 Connection ~ 18400 7900
 Wire Wire Line
-	18400 7900 20800 7900
+	18400 7900 20900 7900
 Wire Wire Line
 	4450 8550 5500 8550
@@
 Connection ~ 18400 8550
 Wire Wire Line
-	18400 8550 20900 8550
+	18400 8550 21000 8550
 Connection ~ 5500 9150
 Wire Wire Line
@@
 	18250 9200 19300 9200
 Wire Wire Line
-	20800 7900 20800 7550
+	20900 7900 20900 6800
 Wire Wire Line
-	20800 7550 21650 7550
+	21000 8550 21000 8100
 Wire Wire Line
-	20900 8550 20900 7750
+	21050 8150 21050 9150
 Wire Wire Line
-	20900 7750 21650 7750
-Wire Wire Line
-	21000 7950 21650 7950
-Wire Wire Line
-	21000 7950 21000 9150
-Wire Wire Line
-	21000 9150 18400 9150
-Wire Wire Line
-	21100 8200 21650 8200
+	21050 9150 18400 9150
 Wire Wire Line
 	21100 8200 21100 9750
@@
 	8550 14900 22800 14900
 Wire Wire Line
-	22800 14900 22800 7300
-Wire Wire Line
-	21650 7550 21650 7450
-Wire Wire Line
-	21650 7450 22750 7450
-Wire Wire Line
-	22750 7450 22750 14850
+	22750 6800 22750 14850
 Wire Wire Line
 	22750 14850 8600 14850
@@
 	8600 13200 22700 13200
 Wire Wire Line
-	22700 13200 22700 7650
-Wire Wire Line
-	22700 7650 21650 7650
+	22700 13200 22700 8100
 Wire Wire Line
-	21650 7650 21650 7750
-Wire Wire Line
-	21650 7950 21650 7850
-Wire Wire Line
-	21650 7850 22650 7850
-Wire Wire Line
-	22650 7850 22650 13150
+	22650 8150 22650 13150
 Wire Wire Line
 	22650 13150 8550 13150
@@
 	8500 13100 22600 13100
 Wire Wire Line
-	22600 13100 22600 8100
-Wire Wire Line
-	22600 8100 21650 8100
+	22600 13100 22600 8200
 Wire Wire Line
-	21650 8100 21650 8200
-Wire Wire Line
-	18400 7300 22800 7300
+	18400 7300 20850 7300
 Wire Wire Line
 	18400 6700 22850 6700
@@
 	3800 5750 3800 9900
 Wire Wire Line
-	12550 5700 22400 5700
+	12550 5350 22400 5350
 Wire Wire Line
-	13900 5650 22350 5650
+	13900 5400 22350 5400
 Wire Wire Line
-	14950 5600 22300 5600
+	14950 5450 22300 5450
 Wire Wire Line
 	16000 5550 22250 5550
 Wire Wire Line
-	18100 5450 22150 5450
+	18100 5650 22150 5650
 Wire Wire Line
-	17050 5500 22200 5500
+	17050 5600 22200 5600
 Wire Wire Line
-	19150 5400 22100 5400
+	19150 5700 22100 5700
 Wire Wire Line
 	3800 5750 11500 5750
@@
 	8000 10200 8000 13350
 Wire Wire Line
-	8000 15700 22100 15700
+	22100 5700 22100 15400
+Wire Wire Line
+	22150 15450 8250 15450
+Wire Wire Line
+	22150 5650 22150 15450
 Wire Wire Line
-	8000 14450 8000 15700
+	22200 5600 22200 15500
 Wire Wire Line
-	22100 5400 22100 15700
+	22250 15550 8150 15550
 Wire Wire Line
-	22150 15650 8050 15650
+	8150 14450 8150 15550
 Wire Wire Line
-	8050 14450 8050 15650
+	22250 5550 22250 15550
 Wire Wire Line
-	22150 5450 22150 15650
+	22300 5450 22300 15650
 Wire Wire Line
-	8100 15600 22200 15600
+	22350 5400 22350 15700
 Wire Wire Line
-	8100 14450 8100 15600
+	22400 5350 22400 15750
 Wire Wire Line
-	22200 5500 22200 15600
+	8000 15750 8000 14450
 Wire Wire Line
-	22250 15550 8150 15550
+	8000 15750 22400 15750
 Wire Wire Line
-	8150 14450 8150 15550
+	8300 14450 8300 15400
 Wire Wire Line
-	22250 5550 22250 15550
+	8300 15400 22100 15400
+Wire Wire Line
+	8050 15700 8050 14450
 Wire Wire Line
-	8200 15500 22300 15500
+	8050 15700 22350 15700
+Wire Wire Line
+	8250 14450 8250 15450
+Wire Wire Line
+	8100 14450 8100 15650
+Wire Wire Line
+	8100 15650 22300 15650
 Wire Wire Line
 	8200 14450 8200 15500
 Wire Wire Line
-	22300 5600 22300 15500
+	8200 15500 22200 15500
 Wire Wire Line
-	22350 15450 8250 15450
+	21050 8150 22650 8150
 Wire Wire Line
-	8250 14450 8250 15450
+	21100 8200 22600 8200
 Wire Wire Line
-	22350 5650 22350 15450
+	20900 6800 22750 6800
 Wire Wire Line
-	22400 15400 8300 15400
+	21000 8100 22700 8100
 Wire Wire Line
-	22400 5700 22400 15400
+	22800 6750 20850 6750
 Wire Wire Line
-	8300 14450 8300 15400
+	20850 6750 20850 7300
+Wire Wire Line
+	22800 6750 22800 14900
 $EndSCHEMATC
